File: tm-feedback/tm-feedback_main.sch (EAGLE design)
At the start: 0 parts

Commit message: Add some intermodule connections
Changed lines of the file:
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@@
 </sheets>
 </module>
-<module name="BLUETOOTH" prefix="" dx="40.64" dy="20.32">
+<module name="BLUETOOTH" prefix="" dx="30.48" dy="20.32">
 <ports>
 <port name="3V3" side="top" coord="0" direction="pwr"/>
@@
 <port name="UART_TX" side="right" coord="-2.54" direction="out"/>
 <port name="UART_RX" side="left" coord="-2.54" direction="in"/>
+<port name="BTN_SIGNAL" side="left" coord="-5.08" direction="in"/>
 </ports>
 <variantdefs>
@@
 <module name="POWER_SUPPLY" prefix="" dx="30.48" dy="20.32">
 <ports>
-<port name="D_3V3" side="bottom" coord="-12.7" direction="pwr"/>
-<port name="D_GND" side="bottom" coord="-7.62" direction="pwr"/>
-<port name="A_3V3" side="bottom" coord="7.62" direction="pwr"/>
-<port name="A_GND" side="bottom" coord="12.7" direction="pwr"/>
+<port name="D_3V3" side="right" coord="7.62" direction="pwr"/>
+<port name="D_GND" side="right" coord="5.08" direction="pwr"/>
+<port name="A_3V3" side="right" coord="-5.08" direction="pwr"/>
+<port name="A_GND" side="right" coord="-7.62" direction="pwr"/>
 </ports>
 <variantdefs>
@@
 </plain>
 <moduleinsts>
-<moduleinst name="MOTOR_DRIVER1" module="MOTOR_DRIVER" x="177.8" y="116.84"/>
-<moduleinst name="MOTOR_DRIVER2" module="MOTOR_DRIVER" x="177.8" y="81.28"/>
-<moduleinst name="BLUETOOTH1" module="BLUETOOTH" x="40.64" y="104.14"/>
-<moduleinst name="MICROCONTROLLER1" module="MICROCONTROLLER" x="104.14" y="104.14"/>
-<moduleinst name="BUTTON1" module="BUTTON" x="104.14" y="66.04"/>
-<moduleinst name="POWER_SUPPLY1" module="POWER_SUPPLY" x="104.14" y="154.94"/>
+<moduleinst name="MOTOR_DRIVER1" module="MOTOR_DRIVER" x="177.8" y="109.22"/>
+<moduleinst name="MOTOR_DRIVER2" module="MOTOR_DRIVER" x="177.8" y="60.96"/>
+<moduleinst name="BLUETOOTH1" module="BLUETOOTH" x="40.64" y="109.22"/>
+<moduleinst name="MICROCONTROLLER1" module="MICROCONTROLLER" x="104.14" y="109.22"/>
+<moduleinst name="BUTTON1" module="BUTTON" x="40.64" y="60.96"/>
+<moduleinst name="POWER_SUPPLY1" module="POWER_SUPPLY" x="104.14" y="160.02"/>
 </moduleinsts>
 <instances>
@@
 </busses>
 <nets>
-</nets>
-</sheet>
+<net name="N$15" class="0">
+<segment>
+<portref moduleinst="MICROCONTROLLER1" port="MOTOR_PWM_1"/>
+<wire x1="129.54" y1="116.84" x2="149.86" y2="116.84" width="0.1524" layer="91"/>
+<wire x1="149.86" y1="116.84" x2="149.86" y2="106.68" width="0.1524" layer="91"/>
+<portref moduleinst="MOTOR_DRIVER1" port="PWM"/>
+<wire x1="149.86" y1="106.68" x2="157.48" y2="106.68" width="0.1524" layer="91"/>
+</segment>
+</net>
+<net name="N$16" class="0">
+<segment>
+<portref moduleinst="MICROCONTROLLER1" port="MOTOR_PWM_2"/>
+<wire x1="129.54" y1="114.3" x2="147.32" y2="114.3" width="0.1524" layer="91"/>
+<wire x1="147.32" y1="114.3" x2="147.32" y2="58.42" width="0.1524" layer="91"/>
+<portref moduleinst="MOTOR_DRIVER2" port="PWM"/>
+<wire x1="147.32" y1="58.42" x2="157.48" y2="58.42" width="0.1524" layer="91"/>
+</segment>
+</net>
+<net name="D_3V3" class="0">
+<segment>
+<portref moduleinst="POWER_SUPPLY1" port="D_3V3"/>
+<wire x1="124.46" y1="167.64" x2="127" y2="167.64" width="0.1524" layer="91"/>
+<label x="127" y="167.64" size="1.778" layer="95"/>
+</segment>
+<segment>
+<portref moduleinst="BLUETOOTH1" port="3V3"/>
+<wire x1="40.64" y1="124.46" x2="40.64" y2="127" width="0.1524" layer="91"/>
+<label x="40.64" y="127" size="1.778" layer="95"/>
+</segment>
+<segment>
+<portref moduleinst="MICROCONTROLLER1" port="3V3"/>
+<wire x1="104.14" y1="124.46" x2="104.14" y2="127" width="0.1524" layer="91"/>
+<label x="104.14" y="127" size="1.778" layer="95"/>
+</segment>
+<segment>
+<portref moduleinst="BUTTON1" port="3V3"/>
+<wire x1="40.64" y1="76.2" x2="40.64" y2="78.74" width="0.1524" layer="91"/>
+<label x="40.64" y="78.74" size="1.778" layer="95"/>
+</segment>
+</net>
+<net name="D_GND" class="0">
+<segment>
+<portref moduleinst="POWER_SUPPLY1" port="D_GND"/>
+<wire x1="124.46" y1="165.1" x2="127" y2="165.1" width="0.1524" layer="91"/>
+<label x="127" y="165.1" size="1.778" layer="95"/>
+</segment>
+<segment>
+<portref moduleinst="BLUETOOTH1" port="GND"/>
+<wire x1="40.64" y1="93.98" x2="40.64" y2="91.44" width="0.1524" layer="91"/>
+<label x="40.64" y="88.9" size="1.778" layer="95"/>
+</segment>
+<segment>
+<portref moduleinst="MICROCONTROLLER1" port="GND"/>
+<wire x1="104.14" y1="93.98" x2="104.14" y2="91.44" width="0.1524" layer="91"/>
+<label x="104.14" y="88.9" size="1.778" layer="95"/>
+</segment>
+<segment>
+<portref moduleinst="BUTTON1" port="GND"/>
+<wire x1="40.64" y1="45.72" x2="40.64" y2="43.18" width="0.1524" layer="91"/>
+<label x="40.64" y="40.64" size="1.778" layer="95"/>
+</segment>
+</net>
+<net name="A_3V3" class="0">
+<segment>
+<portref moduleinst="POWER_SUPPLY1" port="A_3V3"/>
+<wire x1="124.46" y1="154.94" x2="127" y2="154.94" width="0.1524" layer="91"/>
+<label x="127" y="154.94" size="1.778" layer="95"/>
+</segment>
+<segment>
+<portref moduleinst="MOTOR_DRIVER1" port="3V3"/>
+<wire x1="177.8" y1="124.46" x2="177.8" y2="127" width="0.1524" layer="91"/>
+<label x="177.8" y="127" size="1.778" layer="95"/>
+</segment>
+<segment>
+<portref moduleinst="MOTOR_DRIVER2" port="3V3"/>
+<wire x1="177.8" y1="76.2" x2="177.8" y2="78.74" width="0.1524" layer="91"/>
+<label x="177.8" y="78.74" size="1.778" layer="95"/>
+</segment>
+</net>
+<net name="A_GND" class="0">
+<segment>
+<portref moduleinst="POWER_SUPPLY1" port="A_GND"/>
+<wire x1="124.46" y1="152.4" x2="127" y2="152.4" width="0.1524" layer="91"/>
+<label x="127" y="152.4" size="1.778" layer="95"/>
+</segment>
+<segment>
+<portref moduleinst="MOTOR_DRIVER1" port="GND"/>
+<wire x1="177.8" y1="93.98" x2="177.8" y2="91.44" width="0.1524" layer="91"/>
+<label x="177.8" y="88.9" size="1.778" layer="95"/>
+</segment>
+<segment>
+<portref moduleinst="MOTOR_DRIVER2" port="GND"/>
+<wire x1="177.8" y1="45.72" x2="177.8" y2="43.18" width="0.1524" layer="91"/>
+<label x="177.8" y="40.64" size="1.778" layer="95"/>
+</segment>
+</net>
+<net name="N$1" class="0">
+<segment>
+<portref moduleinst="BUTTON1" port="BTN_OUT"/>
+<wire x1="60.96" y1="58.42" x2="71.12" y2="58.42" width="0.1524" layer="91"/>
+<wire x1="71.12" y1="58.42" x2="71.12" y2="104.14" width="0.1524" layer="91"/>
+<portref moduleinst="MICROCONTROLLER1" port="BTN_SIGNAL"/>
+<wire x1="71.12" y1="104.14" x2="78.74" y2="104.14" width="0.1524" layer="91"/>
+</segment>
+</net>
+<net name="N$2" class="0">
+<segment>
+<portref moduleinst="BLUETOOTH1" port="UART_TX"/>
+<portref moduleinst="MICROCONTROLLER1" port="UART_RX"/>
+<wire x1="60.96" y1="106.68" x2="78.74" y2="106.68" width="0.1524" layer="91"/>
+</segment>
+</net>
+</nets>
+</sheet>
