File: tm-feedback/tm-feedback_main.sch (EAGLE design)
At the start: 0 parts

Commit message: Started on PIC schematic
Other:
- note added: "AVDD"
- note added: "AVSS"
- note added: "Decaps C2"
- note added: "Decaps C4"
- note added: "Decaps C5"
- note added: "Decoupling caps"
- note added: "LEDS for debugging"
- note added: "NEED TO WIRE UP"
- note added: "No Cap when programming & debugging"
- note added: "Oscillator"
- note added: "TODO: need to find value"
- note added: "VDD@28"
- note added: "VDD@40"
- note added: "VSS@29"
- note added: "VSS@39"

Commit message: Change PS, add button, remove MOTOR_DRIVER
Parts:
- added MOTOR_DRIVERS, OFF-BOARD_POWER: JST-SMD-2, tactile-music:JST-SMD-2
Connections:
- new net GND: OFF-BOARD_POWER.2
- new net N$3: MOTOR_DRIVERS.1
- new net N$4: MOTOR_DRIVERS.2
- new net N$5: OFF-BOARD_POWER.1
Other:
- note added: "Power switch"
- note added: "Power-on LED"
- note added: "Reverse voltage protection"
- note added: "TACTILE_SWITCH goes here"

Commit message: Wired most of the board up. Currently have ERC issues.
Parts:
- added ANALOG_SENSOR: JST-SMD-2, tactile-music:JST-SMD-2
Connections:
- new net N$15: ANALOG_SENSOR.1
- new net N$16: ANALOG_SENSOR.2
Other:
- note added: "LED Indicators"
- note added: "PICKIT Headers"
- note added: "Pairing LED"
- note added: "UART Headers"
- note removed: "NEED TO WIRE UP"
- moved on the sheet: MOTOR_DRIVERS

Commit message: Replaced JST with picoblade
Parts:
- ANALOG_SENSOR, MOTOR_DRIVERS, OFF-BOARD_POWER: value JST-SMD-2 -> PICOBLADE; device tactile-music:JST-SMD-2 -> tactile-music:PICOBLADE
Changed lines of the file:
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@@
 <part name="R1" library="resistor" deviceset="R-US_" device="R0805" value="60"/>
 <part name="U$1" library="tactile-music" deviceset="MCP1824T-3302E/OT" device=""/>
-<part name="BATTERY" library="tactile-music" deviceset="JST-SMD-2" device=""/>
+<part name="BATTERY" library="tactile-music" deviceset="PICOBLADE" device=""/>
 <part name="U$3" library="tactile-music" deviceset="PMF370XN" device=""/>
 <part name="+3V1" library="supply1" deviceset="+3V3" device=""/>
@@
 <parts>
 <part name="FRAME1" library="frames" deviceset="DINA4_L" device="" value="Top Level"/>
-<part name="OFF-BOARD_POWER" library="tactile-music" deviceset="JST-SMD-2" device=""/>
-<part name="MOTOR_DRIVERS" library="tactile-music" deviceset="JST-SMD-2" device=""/>
+<part name="OFF-BOARD_POWER" library="tactile-music" deviceset="PICOBLADE" device=""/>
+<part name="MOTOR_DRIVERS" library="tactile-music" deviceset="PICOBLADE" device=""/>
 <part name="GND1" library="supply1" deviceset="GND" device=""/>
 <part name="GND2" library="supply1" deviceset="GND" device=""/>
@@
 <part name="+3V3" library="supply1" deviceset="+3V3" device=""/>
 <part name="+3V4" library="supply1" deviceset="+3V3" device=""/>
-<part name="ANALOG_SENSOR" library="tactile-music" deviceset="JST-SMD-2" device=""/>
+<part name="ANALOG_SENSOR" library="tactile-music" deviceset="PICOBLADE" device=""/>
 </parts>
 <sheets>
