File: tm-feedback/tm-feedback_main.sch (EAGLE design)
At the start: 3 parts

Commit message: Add tactile
Other:
- note removed: "TACTILE_SWITCH goes here"
Changed lines of the file:
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@@
 <parts>
 <part name="FRAME1" library="frames" deviceset="DINA4_L" device="" value="Button"/>
-<part name="R1" library="resistor" deviceset="R-US_" device="R0805"/>
+<part name="R1" library="resistor" deviceset="R-US_" device="R0805" value="33k"/>
 <part name="U1" library="tactile-music" deviceset="74AUP1G17GW" device=""/>
-<part name="R2" library="resistor" deviceset="R-US_" device="R0805"/>
+<part name="R2" library="resistor" deviceset="R-US_" device="R0805" value="18k"/>
 <part name="U$1" library="tactile-music" deviceset="DB2S308" device=""/>
-<part name="C1" library="rcl" deviceset="C-EU" device="C0805"/>
+<part name="C1" library="rcl" deviceset="C-EU" device="C0805" value="1uF"/>
 <part name="+3V1" library="supply1" deviceset="+3V3" device=""/>
 <part name="GND1" library="supply1" deviceset="GND" device=""/>
 <part name="+3V2" library="supply1" deviceset="+3V3" device=""/>
 <part name="GND2" library="supply1" deviceset="GND" device=""/>
+<part name="PAIRING_SW" library="tactile-music" deviceset="MC32881_TACTILE" device=""/>
 </parts>
 <sheets>
 <sheet>
 <plain>
-<text x="63.5" y="119.38" size="1.778" layer="98">TACTILE_SWITCH goes here</text>
 </plain>
 <instances>
@@
 <instance part="C1" gate="G$1" x="114.3" y="116.84" rot="R180"/>
 <instance part="+3V1" gate="G$1" x="127" y="134.62"/>
-<instance part="GND1" gate="1" x="127" y="109.22"/>
+<instance part="GND1" gate="1" x="127" y="101.6"/>
 <instance part="+3V2" gate="G$1" x="86.36" y="147.32"/>
-<instance part="GND2" gate="1" x="86.36" y="109.22"/>
+<instance part="GND2" gate="1" x="86.36" y="101.6"/>
+<instance part="PAIRING_SW" gate="G$1" x="86.36" y="116.84" rot="R90"/>
 </instances>
 <busses>
@@
 <pinref part="GND1" gate="1" pin="GND"/>
 <wire x1="129.54" y1="114.3" x2="127" y2="114.3" width="0.1524" layer="91"/>
-<wire x1="127" y1="114.3" x2="127" y2="111.76" width="0.1524" layer="91"/>
+<wire x1="127" y1="114.3" x2="127" y2="104.14" width="0.1524" layer="91"/>
 <label x="124.46" y="114.3" size="1.778" layer="95"/>
 </segment>
 <segment>
 <pinref part="C1" gate="G$1" pin="1"/>
+<wire x1="114.3" y1="114.3" x2="114.3" y2="109.22" width="0.1524" layer="91"/>
 <pinref part="GND2" gate="1" pin="GND"/>
-<wire x1="114.3" y1="114.3" x2="86.36" y2="114.3" width="0.1524" layer="91"/>
-<wire x1="86.36" y1="114.3" x2="86.36" y2="111.76" width="0.1524" layer="91"/>
+<wire x1="114.3" y1="109.22" x2="86.36" y2="109.22" width="0.1524" layer="91"/>
+<wire x1="86.36" y1="109.22" x2="86.36" y2="104.14" width="0.1524" layer="91"/>
+<pinref part="PAIRING_SW" gate="G$1" pin="1"/>
+<wire x1="86.36" y1="109.22" x2="86.36" y2="111.76" width="0.1524" layer="91"/>
+<junction x="86.36" y="109.22"/>
 </segment>
 </net>
@@
 <wire x1="93.98" y1="129.54" x2="86.36" y2="129.54" width="0.1524" layer="91"/>
 <junction x="86.36" y="129.54"/>
+<pinref part="PAIRING_SW" gate="G$1" pin="2"/>
+<wire x1="86.36" y1="121.92" x2="86.36" y2="124.46" width="0.1524" layer="91"/>
+<junction x="86.36" y="124.46"/>
 </segment>
 </net>

Commit message: Arrange PS, rearrange PWM connections for easier layout, rename modules for shorter names (I will try do shorter commits\!)
Parts:
- renumbered OFF-BOARD_POWER to OFF-BOARD_PWR
Other:
- moved on the sheet: MOTOR_DRIVERS

Commit message: More routing
Connections:
- net N$3 renamed PWM_1
- net N$4 renamed PWM_2
- net GND: now also OFF-BOARD_PWR.1; no longer OFF-BOARD_PWR.2
- net N$5: now also OFF-BOARD_PWR.2; no longer OFF-BOARD_PWR.1
Other:
- moved on the sheet: OFF-BOARD_PWR
Changed lines of the file:
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@@
 <instance part="FRAME1" gate="G$1" x="0" y="0"/>
 <instance part="FRAME1" gate="G$2" x="162.56" y="0"/>
-<instance part="OFF-BOARD_PWR" gate="G$1" x="144.78" y="152.4"/>
+<instance part="OFF-BOARD_PWR" gate="G$1" x="144.78" y="152.4" rot="MR180"/>
 <instance part="MOTOR_DRIVERS" gate="G$1" x="152.4" y="121.92" rot="MR180"/>
 <instance part="GND1" gate="1" x="127" y="149.86"/>
@@
 <portref moduleinst="PS" port="GND"/>
 <wire x1="124.46" y1="152.4" x2="127" y2="152.4" width="0.1524" layer="91"/>
-<wire x1="127" y1="152.4" x2="134.62" y2="152.4" width="0.1524" layer="91"/>
-<wire x1="134.62" y1="152.4" x2="134.62" y2="149.86" width="0.1524" layer="91"/>
-<pinref part="OFF-BOARD_PWR" gate="G$1" pin="2"/>
-<wire x1="134.62" y1="149.86" x2="137.16" y2="149.86" width="0.1524" layer="91"/>
 <pinref part="GND1" gate="1" pin="GND"/>
+<wire x1="127" y1="152.4" x2="132.08" y2="152.4" width="0.1524" layer="91"/>
+<wire x1="132.08" y1="152.4" x2="132.08" y2="149.86" width="0.1524" layer="91"/>
 <junction x="127" y="152.4"/>
+<pinref part="OFF-BOARD_PWR" gate="G$1" pin="1"/>
+<wire x1="132.08" y1="149.86" x2="137.16" y2="149.86" width="0.1524" layer="91"/>
 </segment>
 <segment>
@@
 <portref moduleinst="UC" port="BTN_SIGNAL"/>
 <wire x1="76.2" y1="93.98" x2="78.74" y2="93.98" width="0.1524" layer="91"/>
-</segment>
-</net>
-<net name="N$5" class="0">
-<segment>
-<pinref part="OFF-BOARD_PWR" gate="G$1" pin="1"/>
-<portref moduleinst="PS" port="V+"/>
-<wire x1="124.46" y1="154.94" x2="137.16" y2="154.94" width="0.1524" layer="91"/>
 </segment>
 </net>
@@
 </segment>
 </net>
-<net name="N$3" class="0">
+<net name="PWM_1" class="0">
 <segment>
 <pinref part="MOTOR_DRIVERS" gate="G$1" pin="2"/>
@@
 </segment>
 </net>
-<net name="N$4" class="0">
+<net name="PWM_2" class="0">
 <segment>
 <portref moduleinst="UC" port="MOTOR_PWM_2"/>
@@
 </segment>
 </net>
+<net name="N$5" class="0">
+<segment>
+<pinref part="OFF-BOARD_PWR" gate="G$1" pin="2"/>
+<portref moduleinst="PS" port="V+"/>
+<wire x1="124.46" y1="154.94" x2="137.16" y2="154.94" width="0.1524" layer="91"/>
+</segment>
+</net>

Commit message: Even more board layout
Other:
- note added: "Debugging LED"
- note removed: "LEDS for debugging"
